File: HW/dled-esp32-controller.sch (KiCad schematic (older format))
At the start: 40 parts, among them J1 CS_4, J2 CS_3, J3 CS_2, J4 CS_2, J5 CS_3, J6 CS_5, J7 CS_3, J8 CS_Pwr, J9 CS_Pwr, Q1 STD46P4LLF6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

Commit message: Updates some part numbers.
Parts:
- C7: characteristics 10 µF / 16 V / X7R / ESR: 1 mΩ -> 10 µF / 10 V / X5R / ESR: 1 mΩ; part-number EMK212BB7106KG-T -> EMK212BJ106KG-T
- R3, R4: part-number ERJ6ENF2001V -> ERJ-6ENF2201V
- U2: part-number BD48K -> BD48K30G-TL
Changed lines of the file:
@@
 Sheet 1 1
 Title "dled-esp32-controller"
-Date "2019-05-01"
+Date "2019-05-18"
 Rev "15"
 Comp "Calin Radoni"
@@
 F 2 "CalinGeneric:C0805HS" H 4888 4550 50  0001 C CNN
 F 3 "" H 4850 4700 50  0000 C CNN
-F 4 "10 µF / 16 V / X7R / ESR: 1 mΩ" H 0   0   50  0001 C CNN "characteristics"
+F 4 "10 µF / 10 V / X5R / ESR: 1 mΩ" H 0   0   50  0001 C CNN "characteristics"
 F 5 "Taiyo Yuden" H 0   0   50  0001 C CNN "manufacturer"
 F 6 "0805" H 0   0   50  0001 C CNN "package"
-F 7 "EMK212BB7106KG-T" H 0   0   50  0001 C CNN "part-number"
+F 7 "EMK212BJ106KG-T" H 0   0   50  0001 C CNN "part-number"
 	1    4850 4700
 	1    0    0    -1
@@
 F 5 "Panasonic" H 0   0   50  0001 C CNN "manufacturer"
 F 6 "0805" H 0   0   50  0001 C CNN "package"
-F 7 "ERJ6ENF2001V" H 0   0   50  0001 C CNN "part-number"
+F 7 "ERJ-6ENF2201V" H 0   0   50  0001 C CNN "part-number"
 	1    5450 1550
 	-1   0    0    1
@@
 F 5 "Panasonic" H 0   0   50  0001 C CNN "manufacturer"
 F 6 "0805" H 0   0   50  0001 C CNN "package"
-F 7 "ERJ6ENF2001V" H 0   0   50  0001 C CNN "part-number"
+F 7 "ERJ-6ENF2201V" H 0   0   50  0001 C CNN "part-number"
 	1    5650 1550
 	-1   0    0    1
@@
 F 5 "ROHM Semiconductor" H 0   0   50  0001 C CNN "manufacturer"
 F 6 "SSOP3 (SOT23-3)" H 0   0   50  0001 C CNN "package"
-F 7 "BD48K" H 0   0   50  0001 C CNN "part-number"
+F 7 "BD48K30G-TL" H 0   0   50  0001 C CNN "part-number"
 	1    6950 1900
 	1    0    0    -1
